Commit message: Fixed mesh problems, ajusted mesh position, finished IK (it is normalized for the simulation setup, not for the hardware)

File: urdf/hexapod.urdf (robot description, URDF)
Before this commit: robot hexapod_bot, 4 links, 3 joints
Links:
- link base_link: geometry visual mesh filename=package://my_hexapod/meshes/base.stl
- link leg_1_coxa: geometry visual mesh filename=package://my_hexapod/meshes/coxa.stl
- link leg_1_femur: geometry visual mesh filename=package://my_hexapod/meshes/femur.stl
- link leg_1_tibia: geometry visual mesh filename=package://my_hexapod/meshes/tibia.stl
Joints:
- joint joint_1_coxa: axis 0 0 -1 -> 0 0 1; limit lower=0 upper=3.1415 effort=1000 velocity=1.0 -> lower=-1.57 upper=1.57 effort=1000 velocity=1.0; origin xyz=0.1 0.06 0 rpy=0 0 -3.1415 -> xyz=0.0845 0.0668 0 rpy=0 0 0.668
- joint joint_1_femur: limit lower=0 upper=3.1415 effort=1000 velocity=1.0 -> lower=-1.57 upper=1.57 effort=1000 velocity=1.0; origin xyz=0.047 0 0 rpy=0 -1.309 0 -> xyz=0.0464 0 0.015 rpy=0 0 0
- joint joint_1_tibia: limit lower=0 upper=3.1415 effort=1000 velocity=1.0 -> lower=-3.14 upper=3.14 effort=1000 velocity=1.0; origin xyz=0.11 0 0 rpy=0 -0.17 0 -> xyz=0.11 0 0 rpy=0 0 0

Commit message: Create URDF generator, robot config json. Change the IK_node to use the config file. All 6 leg added and the 1-3-5, 2-4-6 configureation programmed. They follow a D shape now

File: urdf/hexapod.urdf (robot description, URDF)
Before this commit: robot hexapod_bot, 4 links, 3 joints
Links:
- added link leg_2_coxa; visual mesh filename=package://my_hexapod/meshes/coxa.stl
- added link leg_2_femur; visual mesh filename=package://my_hexapod/meshes/femur.stl
- added link leg_2_tibia; visual mesh filename=package://my_hexapod/meshes/tibia.stl
- added link leg_3_coxa; visual mesh filename=package://my_hexapod/meshes/coxa.stl
- added link leg_3_femur; visual mesh filename=package://my_hexapod/meshes/femur.stl
- added link leg_3_tibia; visual mesh filename=package://my_hexapod/meshes/tibia.stl
- added link leg_4_coxa; visual mesh filename=package://my_hexapod/meshes/coxa.stl
- added link leg_4_femur; visual mesh filename=package://my_hexapod/meshes/femur.stl
- added link leg_4_tibia; visual mesh filename=package://my_hexapod/meshes/tibia.stl
- added link leg_5_coxa; visual mesh filename=package://my_hexapod/meshes/coxa.stl
- added link leg_5_femur; visual mesh filename=package://my_hexapod/meshes/femur.stl
- added link leg_5_tibia; visual mesh filename=package://my_hexapod/meshes/tibia.stl
- added link leg_6_coxa; visual mesh filename=package://my_hexapod/meshes/coxa.stl
- added link leg_6_femur; visual mesh filename=package://my_hexapod/meshes/femur.stl
- added link leg_6_tibia; visual mesh filename=package://my_hexapod/meshes/tibia.stl
Joints:
- added joint joint_2_coxa: type revolute, parent base_link, child leg_2_coxa, origin xyz=0.0 -0.09259999999999999 0 rpy=0 0 -1.5708, axis 0 0 1, limit lower=-1.57 upper=1.57 effort=1000 velocity=1.0
- added joint joint_2_femur: type revolute, parent leg_2_coxa, child leg_2_femur, origin xyz=0.0464 0 0.015 rpy=0 0 0, axis 0 1 0, limit lower=-1.57 upper=1.57 effort=1000 velocity=1.0
- added joint joint_2_tibia: type revolute, parent leg_2_femur, child leg_2_tibia, origin xyz=0.11 0 -0.0 rpy=0 0 0, axis 0 1 0, limit lower=-3.14 upper=3.14 effort=1000 velocity=1.0
- added joint joint_3_coxa: type revolute, parent base_link, child leg_3_coxa, origin xyz=-0.0852 -0.06720000000000001 0 rpy=0 0 -2.4735, axis 0 0 1, limit lower=-1.57 upper=1.57 effort=1000 velocity=1.0
- added joint joint_3_femur: type revolute, parent leg_3_coxa, child leg_3_femur, origin xyz=0.0464 0 0.015 rpy=0 0 0, axis 0 1 0, limit lower=-1.57 upper=1.57 effort=1000 velocity=1.0
- added joint joint_3_tibia: type revolute, parent leg_3_femur, child leg_3_tibia, origin xyz=0.11 0 -0.0 rpy=0 0 0, axis 0 1 0, limit lower=-3.14 upper=3.14 effort=1000 velocity=1.0
- added joint joint_4_coxa: type revolute, parent base_link, child leg_4_coxa, origin xyz=-0.0852 0.06720000000000001 0 rpy=0 0 2.4735, axis 0 0 1, limit lower=-1.57 upper=1.57 effort=1000 velocity=1.0
- added joint joint_4_femur: type revolute, parent leg_4_coxa, child leg_4_femur, origin xyz=0.0464 0 0.015 rpy=0 0 0, axis 0 1 0, limit lower=-1.57 upper=1.57 effort=1000 velocity=1.0
- added joint joint_4_tibia: type revolute, parent leg_4_femur, child leg_4_tibia, origin xyz=0.11 0 -0.0 rpy=0 0 0, axis 0 1 0, limit lower=-3.14 upper=3.14 effort=1000 velocity=1.0
- added joint joint_5_coxa: type revolute, parent base_link, child leg_5_coxa, origin xyz=0.0 0.09259999999999999 0 rpy=0 0 1.5708, axis 0 0 1, limit lower=-1.57 upper=1.57 effort=1000 velocity=1.0
- added joint joint_5_femur: type revolute, parent leg_5_coxa, child leg_5_femur, origin xyz=0.0464 0 0.015 rpy=0 0 0, axis 0 1 0, limit lower=-1.57 upper=1.57 effort=1000 velocity=1.0
- added joint joint_5_tibia: type revolute, parent leg_5_femur, child leg_5_tibia, origin xyz=0.11 0 -0.0 rpy=0 0 0, axis 0 1 0, limit lower=-3.14 upper=3.14 effort=1000 velocity=1.0
- added joint joint_6_coxa: type revolute, parent base_link, child leg_6_coxa, origin xyz=0.0852 0.06720000000000001 0 rpy=0 0 0.668, axis 0 0 1, limit lower=-1.57 upper=1.57 effort=1000 velocity=1.0
- added joint joint_6_femur: type revolute, parent leg_6_coxa, child leg_6_femur, origin xyz=0.0464 0 0.015 rpy=0 0 0, axis 0 1 0, limit lower=-1.57 upper=1.57 effort=1000 velocity=1.0
- added joint joint_6_tibia: type revolute, parent leg_6_femur, child leg_6_tibia, origin xyz=0.11 0 -0.0 rpy=0 0 0, axis 0 1 0, limit lower=-3.14 upper=3.14 effort=1000 velocity=1.0
- joint joint_1_coxa: origin xyz=0.0845 0.0668 0 rpy=0 0 0.668 -> xyz=0.0852 -0.06720000000000001 0 rpy=0 0 -0.668
- joint joint_1_tibia: origin xyz=0.11 0 0 rpy=0 0 0 -> xyz=0.11 0 -0.0 rpy=0 0 0

Commit message: Talp kapcsolók beépítése, urdf fájl újragenerálása, dimenuiók javítása

File: urdf/hexapod.urdf (robot description, URDF)
Before this commit: robot hexapod_bot, 19 links, 18 joints
Joints:
- joint joint_4_coxa: origin xyz=-0.0852 0.06720000000000001 0 rpy=0 0 2.4735 -> xyz=0.0852 0.06720000000000001 0 rpy=0 0 0.668
- joint joint_6_coxa: origin xyz=0.0852 0.06720000000000001 0 rpy=0 0 0.668 -> xyz=-0.0852 0.06720000000000001 0 rpy=0 0 2.4735

Commit message: Change robot urdf and stl file. Add new base model with the PI and other stuff on it. Chang the dimensions to match the new IRL frame

File: urdf/hexapod.urdf (robot description, URDF)
Before this commit: robot hexapod_bot, 19 links, 18 joints
Joints:
- joint joint_1_coxa: origin xyz=0.0852 -0.06720000000000001 0 rpy=0 0 -0.668 -> xyz=0.0835 0.0665 0 rpy=0 0 0.668
- joint joint_1_femur: origin xyz=0.0464 0 0.015 rpy=0 0 0 -> xyz=0.046799999999999994 0 0.0188 rpy=0 0 0
- joint joint_2_coxa: origin xyz=0.0 -0.09259999999999999 0 rpy=0 0 -1.5708 -> xyz=0.0 0.0916 0 rpy=0 0 1.5708
- joint joint_2_femur: origin xyz=0.0464 0 0.015 rpy=0 0 0 -> xyz=0.046799999999999994 0 0.0188 rpy=0 0 0
- joint joint_3_coxa: origin xyz=-0.0852 -0.06720000000000001 0 rpy=0 0 -2.4735 -> xyz=-0.0835 0.0665 0 rpy=0 0 2.4735
- joint joint_3_femur: origin xyz=0.0464 0 0.015 rpy=0 0 0 -> xyz=0.046799999999999994 0 0.0188 rpy=0 0 0
- joint joint_4_coxa: origin xyz=0.0852 0.06720000000000001 0 rpy=0 0 0.668 -> xyz=0.0835 -0.0665 0 rpy=0 0 -0.668
- joint joint_4_femur: origin xyz=0.0464 0 0.015 rpy=0 0 0 -> xyz=0.046799999999999994 0 0.0188 rpy=0 0 0
- joint joint_5_coxa: origin xyz=0.0 0.09259999999999999 0 rpy=0 0 1.5708 -> xyz=0.0 -0.0916 0 rpy=0 0 -1.5708
- joint joint_5_femur: origin xyz=0.0464 0 0.015 rpy=0 0 0 -> xyz=0.046799999999999994 0 0.0188 rpy=0 0 0
- joint joint_6_coxa: origin xyz=-0.0852 0.06720000000000001 0 rpy=0 0 2.4735 -> xyz=-0.0835 -0.0665 0 rpy=0 0 -2.4735
- joint joint_6_femur: origin xyz=0.0464 0 0.015 rpy=0 0 0 -> xyz=0.046799999999999994 0 0.0188 rpy=0 0 0

Commit message: VIO integrating. Not really working yet

File: urdf/hexapod.urdf (robot description, URDF)
Before this commit: robot hexapod_bot, 19 links, 18 joints
Joints:
- joint joint_1_coxa: origin xyz=0.0835 0.0665 0 rpy=0 0 0.668 -> xyz=0.0835 -0.0665 0 rpy=0 0 -0.668
- joint joint_2_coxa: origin xyz=0.0 0.0916 0 rpy=0 0 1.5708 -> xyz=0.0 -0.0916 0 rpy=0 0 -1.5708
- joint joint_3_coxa: origin xyz=-0.0835 0.0665 0 rpy=0 0 2.4735 -> xyz=-0.0835 -0.0665 0 rpy=0 0 -2.4735
- joint joint_4_coxa: origin xyz=0.0835 -0.0665 0 rpy=0 0 -0.668 -> xyz=0.0835 0.0665 0 rpy=0 0 0.668
- joint joint_5_coxa: origin xyz=0.0 -0.0916 0 rpy=0 0 -1.5708 -> xyz=0.0 0.0916 0 rpy=0 0 1.5708
- joint joint_6_coxa: origin xyz=-0.0835 -0.0665 0 rpy=0 0 -2.4735 -> xyz=-0.0835 0.0665 0 rpy=0 0 2.4735
